File: hardware/kartusche/kartusche.kicad_pcb (KiCad board)
At the start: 2 copper layers, 27.9 x 12.9 mm, 15 parts, among them J10 Conn_01x04_Pin, J1_BOT1 Conn_01x03_Pin, J1_TOP1 Conn_01x03_Pin, J2_BOT1 Conn_01x03_Pin, J2_TOP1 Conn_01x03_Pin, J3_BOT1 Conn_01x03_Pin, J3_TOP1 Conn_01x03_Pin, J7 Conn_01x03_Pin, J8 Conn_01x04_Pin, J9 Conn_01x03_Pin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

Commit message: Base PCB WIP
Parts:
- moved J7 0.64 mm to (110.9, 99.4)
Routing:
- net /G_BOT: track 5.09 -> 6.13 mm
- net /D_BOT: track 5.09 -> 5.73 mm
- net /E_BOT: track 4.01 -> 4.65 mm
