File: hardware/base/base.kicad_pcb (KiCad board)
At the start: 2 copper layers, 109.8 x 41.5 mm, 3 parts

Commit message: Base PCB WIP
Parts:
- removed the REF** at (-37.3, -17.8)
- added C1: 1uF, Capacitor_SMD:C_0805_2012Metric, F.Cu at (1.65, -2.20)
- added C10: 100nF, Capacitor_SMD:C_0402_1005Metric_Pad0.74x0.62mm_HandSolder, F.Cu at (-21.5, 18.9)
- added C11: 100nF, Capacitor_SMD:C_0402_1005Metric_Pad0.74x0.62mm_HandSolder, F.Cu at (-4.40, 19.8)
- added C12: 100nF, Capacitor_SMD:C_0402_1005Metric_Pad0.74x0.62mm_HandSolder, F.Cu at (13.6, 19.9)
- added C13: 100nF, Capacitor_SMD:C_0402_1005Metric_Pad0.74x0.62mm_HandSolder, F.Cu at (24.6, 19.8)
- added C2: 1uF, Capacitor_SMD:C_0805_2012Metric, F.Cu at (31.7, -7.60)
- added C3: 100nF, Capacitor_SMD:C_0402_1005Metric_Pad0.74x0.62mm_HandSolder, B.Cu at (35.1, -17.3)
- added C4: 100nF, Capacitor_SMD:C_0402_1005Metric_Pad0.74x0.62mm_HandSolder, F.Cu at (-5.30, -11.5)
- added C5: 100nF, Capacitor_SMD:C_0402_1005Metric_Pad0.74x0.62mm_HandSolder, F.Cu at (8.53, -9.70)
- added C6: 1uF, Capacitor_SMD:C_0805_2012Metric, F.Cu at (-43.8, -1.30)
- added C7: 1uF, Capacitor_SMD:C_0805_2012Metric, F.Cu at (-3.20, -3.30)
- added C8: 1uF, Capacitor_SMD:C_0805_2012Metric, F.Cu at (18.3, -9.10)
- added C9: 220pF, Capacitor_SMD:C_0402_1005Metric_Pad0.74x0.62mm_HandSolder, F.Cu at (-1.90, 4.60)
- added D1: SOD323, Diode_SMD:D_SOD-323_HandSoldering, F.Cu at (-45.1, -5.15)
- added D2: SOD323, Diode_SMD:D_SOD-323_HandSoldering, F.Cu at (-1.75, 0.70)
- added J1: USB_C_Receptacle_USB2.0, Connector_USB:USB_C_Receptacle_HRO_TYPE-C-31-M-12, F.Cu at (21.0, -16.5)
- added L1: 6.8uH, Inductor_SMD:L_Sunlord_MWSA0402S, F.Cu at (0.80, -5.60)
- added Q1: 2N7002, Package_TO_SOT_SMD:SOT-23, F.Cu at (-41.0, -5.20)
- added Q2: 2N7002, Package_TO_SOT_SMD:SOT-23, F.Cu at (46.5, 4.55)
- added Q3: 2N7002, Package_TO_SOT_SMD:SOT-23, F.Cu at (35.7, 5.90)
- added Q4: 2N7002, Package_TO_SOT_SMD:SOT-23, F.Cu at (41.9, 6.00)
- added R1: 0, Resistor_SMD:R_0402_1005Metric, F.Cu at (27.2, -16.5)
- added R10: 10K, Resistor_SMD:R_0402_1005Metric, F.Cu at (58.2, -1.80)
- added R11: 20, Resistor_SMD:R_0402_1005Metric, F.Cu at (64.1, -6.00)
- added R12: 1M, Resistor_SMD:R_0402_1005Metric, F.Cu at (2.89, 2.90)
- added R13: 22K, Resistor_SMD:R_0402_1005Metric, F.Cu at (-1.90, 3.60)
- added R14: 10K, Resistor_SMD:R_0402_1005Metric, F.Cu at (0.10, 3.70)
- added R15: 20, Resistor_SMD:R_0402_1005Metric, F.Cu at (-36.8, 0.80)
- added R16: 20, Resistor_SMD:R_0402_1005Metric, F.Cu at (-36.8, 2.79)
- added R17: 20, Resistor_SMD:R_0402_1005Metric, F.Cu at (-36.8, 4.78)
- added R2: 5.1K, Resistor_SMD:R_0402_1005Metric, B.Cu at (23.1, -16.5)
- added R3: 5.1K, Resistor_SMD:R_0402_1005Metric, B.Cu at (18.6, -16.0)
- added R4: 22, Resistor_SMD:R_0402_1005Metric, B.Cu at (30.6, -16.4)
- added R5: 22, Resistor_SMD:R_0402_1005Metric, B.Cu at (30.6, -17.8)
- added R6: 10K, Resistor_SMD:R_0402_1005Metric, F.Cu at (58.1, -4.70)
- added R7: 10K, Resistor_SMD:R_0402_1005Metric, F.Cu at (60.7, -4.70)
- added R8: 10K, Resistor_SMD:R_0402_1005Metric, F.Cu at (58.3, 0.10)
- added R9: 10K, Resistor_SMD:R_0402_1005Metric, F.Cu at (60.6, -1.60)
- added SW1: RST, Button_Switch_THT:SW_Tactile_SPST_Angled_PTS645Vx83-2LFS, F.Cu at (-11.1, -17.6)
- added SW2: BOOT, Button_Switch_THT:SW_Tactile_SPST_Angled_PTS645Vx83-2LFS, F.Cu at (6.24, -17.5)
- added U10: TPIC6C595 / TLC6C598, Package_SO:SOIC-16_3.9x9.9mm_P1.27mm, F.Cu at (7.00, 13.2)
- added U11: Kartusche IV9, Flora:Kartusche_IV9, F.Cu at (10.0, 0.87)
- added U12: TPIC6C595 / TLC6C598, Package_SO:SOIC-16_3.9x9.9mm_P1.27mm, F.Cu at (21.5, 13.2)
- added U13: Kartusche IV9, Flora:Kartusche_IV9, F.Cu at (27.0, 0.87)
- added U14: ESP32-C3-MINI-1, PCM_Espressif:ESP32-C3-MINI-1, F.Cu at (38.7, -17.2)
- added U2: LD1117S33TR_SOT223, Package_TO_SOT_SMD:SOT-223-3_TabPin2, F.Cu at (39.0, -3.80)
- added U3: WE-TVS-82400102, Package_TO_SOT_SMD:SOT-23-6, F.Cu at (28.8, -12.6)
- added U4: ~, Flora:MITSUMI_SIQ-02FVS3, F.Cu at (-39.7, -17.6)
- added U5: LMR62421XMF, Package_TO_SOT_SMD:SOT-23-5, F.Cu at (1.55, 0.60)
- added U6: Kartusche IV9, Flora:Kartusche_IV9, F.Cu at (-27.0, 0.87)
- added U7: TPIC6C595 / TLC6C598, Package_SO:SOIC-16_3.9x9.9mm_P1.27mm, F.Cu at (-21.5, 13.2)
- added U8: TPIC6C595 / TLC6C598, Package_SO:SOIC-16_3.9x9.9mm_P1.27mm, F.Cu at (-7.00, 13.2)
- added U9: Kartusche IV9, Flora:Kartusche_IV9, F.Cu at (-10.0, 0.87)
Routing:
- net GND: track 0.00 -> 75.6 mm, vias 0 -> 29
- net +4V: track 0.00 -> 68.8 mm, vias 0 -> 3
- net +5V: track 0.00 -> 52.5 mm
- net +3.3V: track 0.00 -> 26.7 mm, vias 0 -> 1
- net Net-(U6-K6): track 0.00 -> 23.7 mm
- net Net-(U6-K8): track 0.00 -> 22.2 mm
- net Net-(U6-K9): track 0.00 -> 21.6 mm
- net Net-(U6-K7): track 0.00 -> 19.1 mm
- net Net-(U6-K5): track 0.00 -> 19.1 mm
- net Net-(U14-GPIO18/USB_D-): track 0.00 -> 18.0 mm, vias 0 -> 1
- net Net-(U6-K3): track 0.00 -> 16.2 mm
- net Net-(U14-GPIO19/USB_D+): track 0.00 -> 16.0 mm, vias 0 -> 1
- net Net-(J1-D+-PadA6): track 0.00 -> 15.8 mm, vias 0 -> 2
- net Net-(U6-K2): track 0.00 -> 15.8 mm
- net Net-(J1-D--PadA7): track 0.00 -> 15.7 mm
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
Commit message: Minor
Parts:
- moved R8 104.2 mm to (-45.4, -10.4)
- moved R9 103.6 mm to (-42.6, -10.1)
- moved R11 100.7 mm to (-36.6, -6.60)
- moved R10 89.3 mm to (-30.6, -11.3)
- moved R6 68.3 mm to (-9.91, -11.5)
- moved R16 62.6 mm to (24.9, -7.80), turned to 180 degrees
- moved R17 62.6 mm to (24.9, -5.80), turned to 180 degrees
- moved R15 62.1 mm to (24.9, -6.80), turned to 180 degrees
- moved R7 55.0 mm to (6.10, -11.3)
- moved Q2 31.2 mm to (17.0, -5.50)
- moved Q4 24.7 mm to (18.5, -1.90)
- moved Q3 18.5 mm to (21.1, -5.55)
- moved C12 6.71 mm to (7.00, 18.9), turned to 180 degrees
- moved C13 3.07 mm to (21.7, 18.9), turned to 180 degrees
- moved C11 2.66 mm to (-6.90, 18.9), turned to 180 degrees
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Connections:
- Q2 pad 3: Net-(Q2-D) -> /IV9/KB_SINK
- Q3 pad 3: Net-(Q3-D) -> /IV9/KG_SINK
- Q4 pad 3: Net-(Q4-D) -> /IV9/KR_SINK
- U11 pad 13: unconnected-(U11-KB-Pad13) -> /IV9/KB_SINK
- U11 pad 2: unconnected-(U11-KG-Pad2) -> /IV9/KG_SINK
- U11 pad 3: unconnected-(U11-KR-Pad3) -> /IV9/KR_SINK
- U13 pad 13: Net-(Q2-D) -> /IV9/KB_SINK
- U13 pad 2: Net-(Q3-D) -> /IV9/KG_SINK
- U13 pad 3: Net-(Q4-D) -> /IV9/KR_SINK
- U6 pad 13: unconnected-(U6-KB-Pad13) -> /IV9/KB_SINK
- U6 pad 2: unconnected-(U6-KG-Pad2) -> /IV9/KG_SINK
- U6 pad 3: unconnected-(U6-KR-Pad3) -> /IV9/KR_SINK
- U9 pad 13: unconnected-(U9-KB-Pad13) -> /IV9/KB_SINK
- U9 pad 2: unconnected-(U9-KG-Pad2) -> /IV9/KG_SINK
- U9 pad 3: unconnected-(U9-KR-Pad3) -> /IV9/KR_SINK
Routing:
- net /IV9/KB_SINK: track 0.00 -> 105.1 mm, vias 0 -> 5
- net /IV9/KG_SINK: track 0.00 -> 99.3 mm, vias 0 -> 5
- net +3.3V: track 26.7 -> 121.3 mm
- net /IV9/KR_SINK: track 0.00 -> 92.7 mm, vias 0 -> 5
- net /IV9/IV9_SRCK: track 0.00 -> 59.7 mm, vias 0 -> 6
- net /IV9/IV9_~{G1}: track 0.00 -> 56.3 mm, vias 0 -> 4
- net /IV9/IV9_~{CLR}: track 0.00 -> 55.6 mm, vias 0 -> 4
- net /IV9/IV9_SER_IN: track 0.00 -> 52.8 mm, vias 0 -> 1
- net /IV9/IV9_RCK: track 15.6 -> 51.0 mm, vias 1 -> 4
- net Net-(U10-SER_OUT): track 0.00 -> 30.0 mm, vias 0 -> 2
- net Net-(U7-SER_OUT): track 0.00 -> 29.4 mm, vias 0 -> 2
- net Net-(U10-SER_IN): track 0.00 -> 28.7 mm, vias 0 -> 2
- net Net-(U12-DRAIN0): track 0.00 -> 24.8 mm
- net Net-(U10-DRAIN0): track 0.00 -> 22.8 mm
- net Net-(U12-DRAIN2): track 0.00 -> 22.6 mm
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Other:
- board text added: "1"
- board text added: "2"
- board text added: "3"
- board text added: "4"

Commit message: Base V2 Done
Parts:
- added LS1: CMT-8503-85B-SMT-TR, Flora:CMT850385BSMTTR, F.Cu at (-19.1, -14.9)
- moved D1 21.7 mm to (-25.9, -15.2)
- moved C6 20.4 mm to (-25.9, -11.1), turned to -90 degrees
- moved Q1 13.8 mm to (-28.8, -11.6), turned to 90 degrees
- moved R8 10.3 mm to (-35.4, -7.81), turned to -90 degrees
- moved R9 8.63 mm to (-34.3, -7.79), turned to -90 degrees
- moved C5 8.47 mm to (5.00, -19.0), turned to 180 degrees
- moved C4 7.79 mm to (-5.00, -19.0), turned to 180 degrees
- moved R11 6.71 mm to (-31.2, -10.6), turned to -90 degrees
- moved R10 4.35 mm to (-33.2, -7.80), turned to -90 degrees
- moved R6 3.91 mm to (-6.30, -10.0), turned to 180 degrees
- moved SW1 2.67 mm to (-10.4, -15.0)
- moved SW2 2.52 mm to (5.83, -15.0)
- moved R7 2.33 mm to (7.70, -9.60), turned to 180 degrees
- moved U4 0.92 mm to (-40.0, -16.7)
- moved C2 0.60 mm to (31.7, -7.00)
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Connections:
- C4 pad 1: Net-(C4-Pad1) -> /~{RST}
- R11 pad 2: Net-(U14-GPIO20/U0RXD) -> Net-(U14-GPIO21/U0TXD)
- R15 pad 1: /IV9/LED_KG -> /LED_KG
- R16 pad 1: /IV9/LED_KB -> /LED_KB
- R17 pad 1: /IV9/LED_KR -> /LED_KR
- R6 pad 1: Net-(C4-Pad1) -> /~{RST}
- R9 pad 1: Net-(U14-GPIO21/U0TXD) -> Net-(U14-GPIO20/U0RXD)
- SW1 pad 2: Net-(C4-Pad1) -> /~{RST}
- U10 pad 10: /IV9/IV9_RCK -> /LATCH
- U10 pad 15: /IV9/IV9_SRCK -> /SCK
- U10 pad 7: /IV9/IV9_~{CLR} -> /IV9_~{RST}
- U10 pad 8: /IV9/IV9_~{G1} -> /DIM
- U12 pad 10: /IV9/IV9_RCK -> /LATCH
- U12 pad 15: /IV9/IV9_SRCK -> /SCK
- U12 pad 7: /IV9/IV9_~{CLR} -> /IV9_~{RST}
- U12 pad 8: /IV9/IV9_~{G1} -> /DIM
- U14 pad 16: /IV9/LED_KB -> /LATCH
- U14 pad 18: /IV9/IV9_SRCK -> /LED_KR
- U14 pad 19: /IV9/IV9_SER_IN -> /IV9_~{RST}
- U14 pad 20: /IV9/IV9_~{CLR} -> /SCK
- U14 pad 21: /IV9/LED_KR -> /SD
- U14 pad 22: /IV9/LED_KG -> /DIM
- U14 pad 5: /IV9/IV9_~{G1} -> /LED_KB
- U14 pad 6: /IV9/IV9_RCK -> /LED_KG
- U4 pad S: Net-(U14-GPIO21/U0TXD) -> Net-(U14-GPIO20/U0RXD)
- U7 pad 10: /IV9/IV9_RCK -> /LATCH
- U7 pad 15: /IV9/IV9_SRCK -> /SCK
- U7 pad 2: /IV9/IV9_SER_IN -> /SD
- U7 pad 7: /IV9/IV9_~{CLR} -> /IV9_~{RST}
- U7 pad 8: /IV9/IV9_~{G1} -> /DIM
- U8 pad 10: /IV9/IV9_RCK -> /LATCH
- U8 pad 15: /IV9/IV9_SRCK -> /SCK
- U8 pad 7: /IV9/IV9_~{CLR} -> /IV9_~{RST}
- U8 pad 8: /IV9/IV9_~{G1} -> /DIM
Routing:
- net +3.3V: track 121.3 -> 251.5 mm, vias 1 -> 11
- net /LATCH: track 0.00 -> 91.6 mm, vias 0 -> 5
- net /SCK: track 0.00 -> 88.0 mm, vias 0 -> 8
- net Net-(U14-GPIO20/U0RXD): track 12.1 -> 96.5 mm, vias 0 -> 2
- net Net-(U14-GPIO1/ADC1_CH1/XTAL_32K_N): track 0.00 -> 84.0 mm, vias 0 -> 2
- net /DIM: track 0.00 -> 83.9 mm, vias 0 -> 5
- net /SD: track 0.00 -> 81.1 mm, vias 0 -> 2
- net /IV9_~{RST}: track 0.00 -> 80.2 mm, vias 0 -> 5
- net Net-(U14-GPIO0/ADC1_CH0/XTAL_32K_P): track 0.00 -> 73.6 mm, vias 0 -> 2
- net Net-(U14-GPIO21/U0TXD): track 13.2 -> 86.1 mm, vias 0 -> 2
- net +5V: track 53.7 -> 117.3 mm
- net +4V: track 68.8 -> 130.0 mm
- net /IV9/IV9_SRCK: track 59.7 -> 0.00 mm, vias 6 -> 0
- net /IV9/IV9_~{G1}: track 56.3 -> 0.00 mm, vias 4 -> 0
- net /IV9/IV9_~{CLR}: track 55.6 -> 0.00 mm, vias 4 -> 0
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- added copper zone on B.Cu, net GND
- added copper zone on F.Cu, net GND
Other:
- outline, holes or cut-outs redrawn
- board text added: "(c) Yukidamayaki 2023"
- board text added: "CERN-OHL-S"
- board text added: "Flora v2"

Commit message: Minor
Parts:
- added REF**: Fiducial_1.5mm_Mask4.5mm, Fiducial:Fiducial_1.5mm_Mask4.5mm, F.Cu at (-32.6, 10.8)
- added TP1: U0RXD, TestPoint:TestPoint_Pad_D3.0mm, F.Cu at (46.2, -4.80)
- added TP2: U0TXD, TestPoint:TestPoint_Pad_D3.0mm, F.Cu at (46.2, 1.80)
- moved C9 0.20 mm to (-1.90, 4.80)
Routing:
- net Net-(U14-GPIO21/U0TXD): track 86.1 -> 101.9 mm
- net Net-(U14-GPIO20/U0RXD): track 96.5 -> 104.0 mm
- net GND: vias 98 -> 103

Commit message: Base PCB Bugfix
Parts:
- moved D1 13.2 mm to (-18.4, -4.30), turned to 0 degrees
Connections:
- LS1 pad 4: Net-(D1-A) -> unconnected-(LS1---Pad4)
- LS1 pad MP1: unconnected-(LS1-PadMP1) -> Net-(D1-A)
- R4 pad 2: Net-(U14-GPIO19/USB_D+) -> Net-(U14-GPIO18/USB_D-)
- R5 pad 2: Net-(U14-GPIO18/USB_D-) -> Net-(U14-GPIO19/USB_D+)
Routing:
- net Net-(D1-A): track 11.0 -> 23.4 mm
- net +5V: track 117.3 -> 121.3 mm
- net Net-(U14-GPIO19/USB_D+): track 16.0 -> 17.6 mm
- net Net-(U14-GPIO18/USB_D-): track 18.0 -> 17.4 mm
