File: hardware/base/base.kicad_sch (KiCad schematic)
At the start: 36 parts, among them J1 USB_C_Receptacle_USB2.0, Q1 2N7002, SW1 RST, SW2 BOOT, U1 ESP32-C3-WROOM-02, U2 LD1117S33TR_SOT223, U3 WE-TVS-82400102, U5 LMR62421XMF

Commit message: Base PCB WIP
Parts:
- removed U1: ESP32-C3-WROOM-02, PCM_Espressif:ESP32-C3-WROOM-02, symbol PCM_Espressif:ESP32-C3-WROOM-02
- added U14: ESP32-C3-MINI-1, PCM_Espressif:ESP32-C3-MINI-1, symbol PCM_Espressif:ESP32-C3-MINI-1
- SW1, SW2: footprint (none) -> Button_Switch_THT:SW_Tactile_SPST_Angled_PTS645Vx83-2LFS
- U4: footprint (none) -> Flora:MITSUMI_SIQ-02FVS3
Connections:
- net +3.3V: now also U14.3 (3V3); no longer C6.1, D1.1 (K), LS1.1
- net +5V: now also C6.1, D1.1 (K), LS1.1
- net GND: now also U14.1 (GND), U14.11 (GND), U14.14 (GND), U14.2 (GND), U14.36 (GND), U14.37 (GND), U14.38 (GND), U14.39 (GND), U14.40 (GND), U14.41 (GND), U14.42 (GND), U14.43 (GND), U14.44 (GND), U14.45 (GND), U14.46 (GND), U14.47 (GND), U14.48 (GND), U14.49 (GND), U14.50 (GND), U14.51 (GND), U14.52 (GND), U14.53 (GND)
- net IV9/IV9_RCK: now also U14.6 (GPIO3/ADC1_CH3)
- net IV9/IV9_SER_IN: now also U14.19 (GPIO5/ADC2_CH0)
- net IV9/IV9_SRCK: now also U14.18 (GPIO4/ADC1_CH4)
- net IV9/IV9_~{CLR}: now also U14.20 (GPIO6)
- net IV9/IV9_~{G1}: now also U14.5 (GPIO2/ADC1_CH2)
- net IV9/LED_KB: now also U14.16 (GPIO10)
- net IV9/LED_KG: now also U14.22 (GPIO8)
- net IV9/LED_KR: now also U14.21 (GPIO7)
- net ~{BOOT}: now also U14.23 (GPIO9)
- net ~{RST}: now also U14.8 (EN/CHIP_PU)
- net at R9.1, U4.S (Sw): now also U14.31 (GPIO21/U0TXD)
- net at R10.1, U4.B: now also U14.12 (GPIO0/ADC1_CH0/XTAL_32K_P)
- net at R5.2: now also U14.26 (GPIO18/USB_D-)
- net at R8.1, U4.A: now also U14.13 (GPIO1/ADC1_CH1/XTAL_32K_N)
- net at R4.2: now also U14.27 (GPIO19/USB_D+)
- net at R11.2: now also U14.30 (GPIO20/U0RXD)

Commit message: Base V2 Done
Parts:
- removed LS1: Speaker, symbol Device:Speaker
- added LS1: CMT-8503-85B-SMT-TR, CMT850385BSMTTR, symbol Flora:CMT-8503-85B-SMT-TR
Connections:
- net +5V: now also LS1.1 (+)
- net ~{RST}: now also C4.1, R6.1, SW1.2
- net at R9.1, U4.S (Sw): now also U14.30 (GPIO20/U0RXD); no longer U14.31 (GPIO21/U0TXD)
- net at D1.2 (A), Q1.3 (D): now also LS1.4 (-)
- net at R11.2: now also U14.31 (GPIO21/U0TXD); no longer U14.30 (GPIO20/U0RXD)
- net IV9/IV9_RCK renamed LED_KG
- net IV9/IV9_SER_IN renamed IV9_~{RST}
- net IV9/IV9_SRCK renamed LED_KR
- net IV9/IV9_~{CLR} renamed SCK
- net IV9/IV9_~{G1} renamed LED_KB
- net IV9/LED_KB renamed LATCH
- net IV9/LED_KG renamed DIM
- net IV9/LED_KR renamed SD
- no-connect marks 3 -> 5

Commit message: Minor
Parts:
- added TP1: U0RXD, TestPoint:TestPoint_Pad_D3.0mm, symbol Connector:TestPoint
- added TP2: U0TXD, TestPoint:TestPoint_Pad_D3.0mm, symbol Connector:TestPoint
Connections:
- net at R9.1, U14.30 (GPIO20/U0RXD), U4.S (Sw): now also TP1.1
- net at R11.2, U14.31 (GPIO21/U0TXD): now also TP2.1
Changed lines of the file:
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@@
   (junction (at 110.49 160.02) (diameter 0) (color 0 0 0 0)
   )
+  (junction (at 161.29 69.85) (diameter 0) (color 0 0 0 0)
+  )
   (junction (at 73.66 67.31) (diameter 0) (color 0 0 0 0)
   )
@@
   )
   (junction (at 77.47 102.87) (diameter 0) (color 0 0 0 0)
+  )
+  (junction (at 156.21 72.39) (diameter 0) (color 0 0 0 0)
   )
   (junction (at 52.07 67.31) (diameter 0) (color 0 0 0 0)
@@
     (stroke (width 0) (type default))
   )
+  (wire (pts (xy 161.29 69.85) (xy 163.83 69.85))
+    (stroke (width 0) (type default))
+  )
   (wire (pts (xy 220.98 142.24) (xy 224.79 142.24))
     (stroke (width 0) (type default))
@@
     (stroke (width 0) (type default))
   )
-  (wire (pts (xy 162.56 41.91) (xy 162.56 69.85))
+  (wire (pts (xy 161.29 41.91) (xy 161.29 69.85))
     (stroke (width 0) (type default))
   )
@@
     (stroke (width 0) (type default))
   )
-  (wire (pts (xy 157.48 41.91) (xy 162.56 41.91))
+  (wire (pts (xy 157.48 41.91) (xy 161.29 41.91))
     (stroke (width 0) (type default))
   )
@@
     (stroke (width 0) (type default))
   )
+  (wire (pts (xy 156.21 72.39) (xy 163.83 72.39))
+    (stroke (width 0) (type default))
+  )
   (wire (pts (xy 222.25 62.23) (xy 217.17 62.23))
     (stroke (width 0) (type default))
@@
     (stroke (width 0) (type default))
   )
-  (wire (pts (xy 152.4 69.85) (xy 162.56 69.85))
+  (wire (pts (xy 152.4 69.85) (xy 161.29 69.85))
     (stroke (width 0) (type default))
   )
@@
         (path "/22dc2c6c-1801-4d51-b98c-8b9b53e66a91"
           (reference "#PWR06") (unit 1)
+        )
+      )
+    )
+  )
+  (symbol (lib_id "Connector:TestPoint") (at 163.83 69.85 270) (unit 1)
+    (in_bom yes) (on_board yes) (dnp no)
+    (property "Reference" "TP2" (at 168.91 69.85 90)
+      (effects (font (size 1.27 1.27)) (justify left))
+    )
+    (property "Value" "U0TXD" (at 173.99 69.85 90)
+      (effects (font (size 1.27 1.27)) (justify left))
+    )
+    (property "Footprint" "TestPoint:TestPoint_Pad_D3.0mm" (at 163.83 74.93 0)
+      (effects (font (size 1.27 1.27)) hide)
+    )
+    (property "Datasheet" "~" (at 163.83 74.93 0)
+      (effects (font (size 1.27 1.27)) hide)
+    )
+    (pin "1")
+    (instances
+      (project "base"
+        (path "/22dc2c6c-1801-4d51-b98c-8b9b53e66a91"
+          (reference "TP2") (unit 1)
         )
       )
@@
         )
       )
+    )
+  )
+  (symbol (lib_id "Connector:TestPoint") (at 163.83 72.39 270) (unit 1)
+    (in_bom yes) (on_board yes) (dnp no)
+    (property "Reference" "TP1" (at 168.91 72.39 90)
+      (effects (font (size 1.27 1.27)) (justify left))
+    )
+    (property "Value" "U0RXD" (at 173.99 72.39 90)
+      (effects (font (size 1.27 1.27)) (justify left))
+    )
+    (property "Footprint" "TestPoint:TestPoint_Pad_D3.0mm" (at 163.83 77.47 0)
+      (effects (font (size 1.27 1.27)) hide)
+    )
+    (property "Datasheet" "~" (at 163.83 77.47 0)
+      (effects (font (size 1.27 1.27)) hide)
+    )
+    (pin "1")
+    (instances
+      (project "base"
+        (path "/22dc2c6c-1801-4d51-b98c-8b9b53e66a91"
+          (reference "TP1") (unit 1)
+        )
+      )

Commit message: Base PCB Bugfix
Connections:
- net at R5.2: now also U14.27 (GPIO19/USB_D+); no longer U14.26 (GPIO18/USB_D-)
- net at D1.2 (A), Q1.3 (D): now also LS1.MP1; no longer LS1.4 (-)
- net at R4.2: now also U14.26 (GPIO18/USB_D-); no longer U14.27 (GPIO19/USB_D+)
Changed lines of the file:
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@@
   (no_connect (at 222.25 90.17))
   (no_connect (at 224.79 142.24))
-  (no_connect (at 114.3 29.21))
   (no_connect (at 222.25 92.71))
+  (no_connect (at 137.16 31.75))
   (wire (pts (xy 187.96 74.93) (xy 194.31 74.93))
     (stroke (width 0) (type default))
@@
     (stroke (width 0) (type default))
   )
-  (wire (pts (xy 152.4 77.47) (xy 176.53 77.47))
-    (stroke (width 0) (type default))
-  )
   (wire (pts (xy 179.07 58.42) (xy 179.07 62.23))
     (stroke (width 0) (type default))
@@
     (stroke (width 0) (type default))
   )
+  (wire (pts (xy 111.76 29.21) (xy 114.3 29.21))
+    (stroke (width 0) (type default))
+  )
+  (wire (pts (xy 152.4 80.01) (xy 173.99 80.01))
+    (stroke (width 0) (type default))
+  )
   (wire (pts (xy 171.45 95.25) (xy 171.45 149.86))
     (stroke (width 0) (type default))
@@
     (stroke (width 0) (type default))
   )
+  (wire (pts (xy 176.53 80.01) (xy 182.88 80.01))
+    (stroke (width 0) (type default))
+  )
   (wire (pts (xy 52.07 63.5) (xy 52.07 67.31))
     (stroke (width 0) (type default))
@@
     (stroke (width 0) (type default))
   )
+  (wire (pts (xy 176.53 77.47) (xy 173.99 80.01))
+    (stroke (width 0) (type default))
+  )
   (wire (pts (xy 52.07 73.66) (xy 52.07 77.47))
     (stroke (width 0) (type default))
@@
     (stroke (width 0) (type default))
   )
-  (wire (pts (xy 139.7 31.75) (xy 139.7 35.56))
-    (stroke (width 0) (type default))
-  )
   (wire (pts (xy 144.78 34.29) (xy 144.78 35.56))
     (stroke (width 0) (type default))
@@
     (stroke (width 0) (type default))
   )
+  (wire (pts (xy 152.4 77.47) (xy 173.99 77.47))
+    (stroke (width 0) (type default))
+  )
   (wire (pts (xy 52.07 77.47) (xy 52.07 80.01))
     (stroke (width 0) (type default))
@@
     (stroke (width 0) (type default))
   )
+  (wire (pts (xy 176.53 80.01) (xy 173.99 77.47))
+    (stroke (width 0) (type default))
+  )
   (wire (pts (xy 99.06 160.02) (xy 110.49 160.02))
     (stroke (width 0) (type default))
@@
     (stroke (width 0) (type default))
   )
-  (wire (pts (xy 139.7 35.56) (xy 144.78 35.56))
+  (wire (pts (xy 111.76 35.56) (xy 144.78 35.56))
+    (stroke (width 0) (type default))
+  )
+  (wire (pts (xy 111.76 35.56) (xy 111.76 29.21))
     (stroke (width 0) (type default))
   )
@@
     (stroke (width 0) (type default))
   )
-  (wire (pts (xy 137.16 31.75) (xy 139.7 31.75))
-    (stroke (width 0) (type default))
-  )
   (wire (pts (xy 80.01 114.3) (xy 80.01 124.46))
     (stroke (width 0) (type default))
@@
     (stroke (width 0) (type default))
   )
-  (wire (pts (xy 152.4 80.01) (xy 182.88 80.01))
-    (stroke (width 0) (type default))
-  )
